File: hardware/dandelion/dandelion.sch (KiCad schematic (older format))
At the start: 97 parts, among them J1 PCB Antenna, J2 USB-MICRO-B, P1 DIGITAL, P10 GIO6, P11 DCLK, P12 DIO, P2 PROGRAM, P3 JTAG, P4 EXPAND, P5 ANALOG, P6 VCC, P7 VBUS, P8 1V8, P9 GIO1, Q1 PDTA123Y, Q2 MOSFET_P, SW1 SW_PUSH, U1 TC1184, U2 PT7M8206, U3 CC2400, U4 LPC175X, X1 XCVR XTAL

Commit message: Dandelion: folded dipole PCB antenna
Parts:
- removed C1: 5p6, symbol C
- removed C3, C4: 0p5, symbol C
- removed C5: 100nF, symbol C
- removed J1: PCB Antenna, symbol BNC
- removed L2, L3: 7n5, symbol INDUCTOR
- added J1: PCB antenna, symbol GSG-FOLDED-DIPOLE
- L1: value 5n6 -> 12nH; Field2 L-07C5N6SV6T -> L-07C12NJV6T; Field3 CER INDUCTOR 5.6NH 0402 -> CER INDUCTOR 12NH 0402
Connections:
- wire segments 368 -> 359
Other:
- moved on the sheet: L4

Commit message: Dandelion: added R8C
Parts:
- added C? (x2): 100nF, 0603, symbol C
- added C?: 10µF, 0603, symbol C
- added D?: DIODESCH, symbol DIODESCH
- added P?: E8A, symbol CONN_4
- added P?: R8C PROGRAM, 100MIL-HEADER-1X6-EDGE, symbol CONN_6
- added P?: PCB JUMPER, symbol CONN_2
- added P?: R8C EXPAND, symbol CONN_10
- added R? (x2): 4k7, 0603, symbol R
- added U?: R5F212L4SNFP, symbol GSG-R8C/2K/2L
- P2: value PROGRAM -> LPC PROGRAM
Connections:
- net labels added: CC1V8, CC3V3, MISO, MOSI, P0_0, P4_2, P4_5, SCK, XIN, XOUT
- net labels removed: RX, TX
- wire segments 359 -> 508
- no-connect marks 16 -> 18
Other:
- note added: "R8C expansion port\nmostly pins that can be\nrepurposed if LPC175x\nis not installed"
- moved on the sheet: BT1, C10, C11, C12, C13, C14, C15, C16, C17, C18, C19, C2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

Commit message: Dandelion: designated factory installed portions on schematic
Parts:
- removed R?: 4k7, 0603, symbol R
- added R?: 10k, 0603, symbol R
- D14, D17: Field4 DNP -> (none)
Connections:
- wire segments 508 -> 428
Other:
- note added: "LPC175x\nprogramming\nconnector"
- note added: "factory install"
- note added: "if installing power\nswitching circuit, cut\nPCB JUMPER above"
- note removed: "D14 not populated\n(to save power)"
- note removed: "D17 not populated\n(to save power)"
- note removed: "programming\n connector"
- moved on the sheet: BT1, C11, C16, P?, R23, U2

Commit message: Dandelion: DNP/DIY designations
Parts:
- C13, C14, C2, C20, C21, C25, C26, C27, C28, C29, C30, C33, C34, D14, D15, D16, D17, J2, Q1, Q2, R1, R10, R12, R13, R15, R16, R24, R8, R9, U1, U4: Field4 (none) -> DIY
- C15: Field4 (none) -> DNP
- J1: Field1 DNP -> (none); Field4 (none) -> DNP
- P1, P10, P11, P12, P2, P3, P4, P5, P6, P7, P8, P9: Field3 DNP -> (none); Field4 (none) -> DNP
- P13: renamed from P?; Field4 (none) -> DNP
- P15, P16: renamed from P?; Field3 DNP -> (none); Field4 (none) -> DNP
- gave numbers to parts that had none: 8
Other:
- note added: "3V supply (VCC) switches between battery and\nUSB power depending on bus power availability"
- note added: "C4 optional\nfor ADC"
- note added: "Field4 in component properties indicates:\n\nDIY: Do It Yourself parts to be\ninstalled by user for\nUbertooth function\n\nDNP: Do Not Populate optional\nparts not needed for Ubertooth\nfunction or built in to PCB\n\nnone: installed at factory"
- note removed: "3V supply switches between battery and USB\npower depending on bus power availability"

Commit message: Dandelion: component selection
Parts:
- removed C2: 470pF, symbol C
- removed D16: BAW56, symbol BAW56
- removed U1: TC1184, symbol SI9183-A
- added C?: 10µF, symbol C
- added D?: DIODESCH, symbol DIODESCH
- added U?: NCP502, symbol TCR5SB
- C1: footprint 0603 -> (none); Field1 (none) -> TDK; Field2 (none) -> C3216Y5V1A106ZT/1.15; Field3 (none) -> Multilayer Ceramic Capacitors (MLCC) - SMD/SMT 1206 10uF 10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
- C15: Field1 Panasonic -> Nichon; Field2 EEE-1AA101WR -> UUR1C101MCL1GS; Field3 CAP ALUM 100UF 10V 20% SMD -> Aluminum Electrolytic Capacitors - SMD 16volts 100uF 20% 85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
- D18: Field1 (none) -> Fairchild; Field2 (none) -> RB521S30; Field3 (none) -> DIODE SCHOTTKY 30V 200MA SOD523F
- P14: Field4 (none) -> DNP
- R11, R14, R17, R18, R19, R2, R20, R21, R3, R4, R5, R6, R7: value 330 -> 150; Field1 Bourns -> Panasonic-ECG; Field2 CR0603-JW-331ELF -> ERJ-3GEYJ151V; Field3 Thick Film Resistors - SMD 0603 330OHMS 5% 1/10WATT -> RES 150 OHM 1/10W 5% 0603 SMD
- R26: Field1 (none) -> Panasonic-ECG; Field2 (none) -> ERJ-3GEYJ472V; Field3 (none) -> RES 4.7K OHM 1/10W 5% 0603 SMD
- SW1: Field1 TE Connectivity -> APEM Components; Field2 FSM4JSMATR -> ADTSM62RVTR; Field3 SWITCH TACT MINI 6X6MM SMD GW -> SWITCH TACT SPST 12VDC 260GF
- U5: Field1 (none) -> Renesas; Field2 (none) -> R5F212L4SNFP#U0; Field3 (none) -> IC R8C/2L MCU FLASH 32LQFP
Connections:
- wire segments 428 -> 429
- no-connect marks 18 -> 17
Other:
- moved on the sheet: C15, C25, C29, R1

Commit message: Dandelion: LED series resistors upped to 220 ohm so as not to exceed R8C/2L i/o pin current rating
Parts:
- R11, R14, R17, R18, R19, R2, R20, R21, R3, R4, R5, R6, R7: value 150 -> 220; Field2 ERJ-3GEYJ151V -> ERJ-3GEYJ221V; Field3 RES 150 OHM 1/10W 5% 0603 SMD -> RES 220 OHM 1/10W 5% 0603 SMD
- gave numbers to parts that had none: 3
Connections:
- no-connect marks 17 -> 27

Commit message: Dandelion: changed R8C PROGRAM connector so that it will (hopefully) work with SparkFun FTDI board
Connections:
- net at P14.1 (P1), R25.1, U5.3 (RESET): now also P15.6; no longer P15.2
Other:
- note added: "supplied power not\nto exceed 3.3V"

Commit message: Dandelion: minor BOM corrections
Parts:
- C15: Field1 Nichon -> Nichicon
- U1: Field4 (none) -> DIY
Changed lines of the file:
@@
-EESchema Schematic File Version 2  date Sat 27 Aug 2011 03:46:44 PM MDT
+EESchema Schematic File Version 2  date Sat 27 Aug 2011 03:56:37 PM MDT
 LIBS:ubertooth-symbols
 LIBS:power
@@
 F 5 "NCP502SQ35T2G" H 2250 9050 60  0001 C CNN "Field2"
 F 6 "IC REG VOLTAGE 180MA 3.5V SC70-6" H 2250 9050 60  0001 C CNN "Field3"
+F 7 "DIY" H 2250 9050 60  0001 C CNN "Field4"
 	1    2250 9050
 	1    0    0    -1
@@
 F 0 "C15" H 4200 9950 50  0000 L CNN
 F 1 "100µF" H 4200 9750 50  0000 L CNN
-F 4 "Nichon" H 4150 9850 60  0001 C CNN "Field1"
+F 4 "Nichicon" H 4150 9850 60  0001 C CNN "Field1"
 F 5 "UUR1C101MCL1GS" H 4150 9850 60  0001 C CNN "Field2"
 F 6 "Aluminum Electrolytic Capacitors - SMD 16volts 100uF 20% 85C 8X6.2" H 4150 9850 60  0001 C CNN "Field3"
